Commit message: [add] option to switch between 2D RPLiDAR and 3D GPU LiDAR at launch time

File: turtlebot4/turtlebot4_description/urdf/standard/turtlebot4.urdf.xacro (robot description, xacro)
@@ -4,4 +4,5 @@
   <xacro:include filename="$(find irobot_create_description)/urdf/create3.urdf.xacro" />
   <xacro:include filename="$(find turtlebot4_description)/urdf/sensors/rplidar.urdf.xacro" />
+  <xacro:include filename="$(find turtlebot4_description)/urdf/sensors/gpu_lidar.urdf.xacro" />
   <xacro:include filename="$(find turtlebot4_description)/urdf/sensors/oakd.urdf.xacro" />
   <xacro:include filename="$(find turtlebot4_description)/urdf/sensors/camera_bracket.urdf.xacro" />
@@ -91,8 +92,16 @@
   </xacro:tower_sensor_plate>
   <!-- Turtlebot4 sensor definitions -->
-  <xacro:rplidar name="rplidar" parent_link="shell_link" gazebo="$(arg gazebo)">
-    <origin xyz="${rplidar_x_offset} ${rplidar_y_offset} ${rplidar_z_offset}"
-            rpy="0 0 ${pi/2}"/>
-  </xacro:rplidar>
+  <xacro:if value="$(arg use_gpu_lidar)">
+    <xacro:gpu_lidar name="rplidar" parent_link="shell_link" gazebo="$(arg gazebo)">
+      <origin xyz="${rplidar_x_offset} ${rplidar_y_offset} ${rplidar_z_offset}"
+              rpy="0 0 ${pi/2}"/>
+    </xacro:gpu_lidar>
+  </xacro:if>
+  <xacro:unless value="$(arg use_gpu_lidar)">
+    <xacro:rplidar name="rplidar" parent_link="shell_link" gazebo="$(arg gazebo)">
+      <origin xyz="${rplidar_x_offset} ${rplidar_y_offset} ${rplidar_z_offset}"
+              rpy="0 0 ${pi/2}"/>
+    </xacro:rplidar>
+  </xacro:unless>
   <xacro:camera_bracket name="oakd_camera_bracket">
     <origin xyz="${camera_mount_x_offset} ${camera_mount_y_offset} ${camera_mount_z_offset}"/>

Commit message: [temp] not working Velodyne

File: turtlebot4/turtlebot4_description/urdf/standard/turtlebot4.urdf.xacro (robot description, xacro)
@@ -5,4 +5,5 @@
   <xacro:include filename="$(find turtlebot4_description)/urdf/sensors/rplidar.urdf.xacro" />
   <xacro:include filename="$(find turtlebot4_description)/urdf/sensors/gpu_lidar.urdf.xacro" />
+  <xacro:include filename="$(find turtlebot4_description)/urdf/sensors/velodyne.urdf.xacro" />
   <xacro:include filename="$(find turtlebot4_description)/urdf/sensors/oakd.urdf.xacro" />
   <xacro:include filename="$(find turtlebot4_description)/urdf/sensors/camera_bracket.urdf.xacro" />
@@ -98,9 +99,17 @@
     </xacro:gpu_lidar>
   </xacro:if>
+  <xacro:if value="$(arg use_velodyne_lidar)">
+    <xacro:velodyne name="velodyne" parent_link="shell_link" gazebo="$(arg gazebo)">
+      <origin xyz="${rplidar_x_offset} ${rplidar_y_offset} ${rplidar_z_offset}"
+              rpy="0 0 0"/>
+    </xacro:velodyne>
+  </xacro:if>
   <xacro:unless value="$(arg use_gpu_lidar)">
-    <xacro:rplidar name="rplidar" parent_link="shell_link" gazebo="$(arg gazebo)">
-      <origin xyz="${rplidar_x_offset} ${rplidar_y_offset} ${rplidar_z_offset}"
-              rpy="0 0 ${pi/2}"/>
-    </xacro:rplidar>
+    <xacro:unless value="$(arg use_velodyne_lidar)">
+      <xacro:rplidar name="rplidar" parent_link="shell_link" gazebo="$(arg gazebo)">
+        <origin xyz="${rplidar_x_offset} ${rplidar_y_offset} ${rplidar_z_offset}"
+                rpy="0 0 ${pi/2}"/>
+      </xacro:rplidar>
+    </xacro:unless>
   </xacro:unless>
   <xacro:camera_bracket name="oakd_camera_bracket">

Commit message: Revert "[temp] not working Velodyne"
This reverts commit 4496e1bc45dfd8790ac376dc758bf931c829226c.

File: turtlebot4/turtlebot4_description/urdf/standard/turtlebot4.urdf.xacro (robot description, xacro)
@@ -5,5 +5,4 @@
   <xacro:include filename="$(find turtlebot4_description)/urdf/sensors/rplidar.urdf.xacro" />
   <xacro:include filename="$(find turtlebot4_description)/urdf/sensors/gpu_lidar.urdf.xacro" />
-  <xacro:include filename="$(find turtlebot4_description)/urdf/sensors/velodyne.urdf.xacro" />
   <xacro:include filename="$(find turtlebot4_description)/urdf/sensors/oakd.urdf.xacro" />
   <xacro:include filename="$(find turtlebot4_description)/urdf/sensors/camera_bracket.urdf.xacro" />
@@ -99,17 +98,9 @@
     </xacro:gpu_lidar>
   </xacro:if>
-  <xacro:if value="$(arg use_velodyne_lidar)">
-    <xacro:velodyne name="velodyne" parent_link="shell_link" gazebo="$(arg gazebo)">
+  <xacro:unless value="$(arg use_gpu_lidar)">
+    <xacro:rplidar name="rplidar" parent_link="shell_link" gazebo="$(arg gazebo)">
       <origin xyz="${rplidar_x_offset} ${rplidar_y_offset} ${rplidar_z_offset}"
-              rpy="0 0 0"/>
-    </xacro:velodyne>
-  </xacro:if>
-  <xacro:unless value="$(arg use_gpu_lidar)">
-    <xacro:unless value="$(arg use_velodyne_lidar)">
-      <xacro:rplidar name="rplidar" parent_link="shell_link" gazebo="$(arg gazebo)">
-        <origin xyz="${rplidar_x_offset} ${rplidar_y_offset} ${rplidar_z_offset}"
-                rpy="0 0 ${pi/2}"/>
-      </xacro:rplidar>
-    </xacro:unless>
+              rpy="0 0 ${pi/2}"/>
+    </xacro:rplidar>
   </xacro:unless>
   <xacro:camera_bracket name="oakd_camera_bracket">
